Commit message: working viewer

File: frontend/public/models/kuka.urdf (robot description, URDF)
Before this commit: robot lbr_iiwa7_r800, 8 links, 7 joints
Links:
- link base_link: geometry collision mesh filename=/public/models/meshes/base_link.STL; visual mesh filename=/public/models/meshes/base_link.DAE
- link link1: geometry collision mesh filename=/public/models/meshes/link1.STL; visual mesh filename=/public/models/meshes/link1.DAE
- link link2: geometry collision mesh filename=/public/models/meshes/link2.STL; visual mesh filename=/public/models/meshes/link2.DAE
- link link3: geometry collision mesh filename=/public/models/meshes/link3.STL; visual mesh filename=/public/models/meshes/link3.DAE
- link link4: geometry collision mesh filename=/public/models/meshes/link4.STL; visual mesh filename=/public/models/meshes/link4.DAE
- link link5: geometry collision mesh filename=/public/models/meshes/link5.STL; visual mesh filename=/public/models/meshes/link5.DAE
- link link6: geometry collision mesh filename=/public/models/meshes/link6.STL; visual mesh filename=/public/models/meshes/link6.DAE
- link link7: geometry collision mesh filename=/public/models/meshes/link7.STL; visual mesh filename=/public/models/meshes/link7.DAE
